Commit message: Update xacro to match urdf

File: urdf/adeept_awr.urdf.xacro (robot description, xacro)
@@ -1,151 +1,165 @@
 <?xml version="1.0"?>
-<robot name="adeept_awr">
+<robot xmlns:xacro="http://ros.org/wiki/xacro" name="adeept_awr">
+  <!-- Variables for chassis -->
+  <xacro:property name="c_len_x" value="0.13"/>
+  <xacro:property name="c_len_y" value="0.12"/>
+  <xacro:property name="c_len_z" value="0.08"/>
+  <xacro:property name="c_mass" value="0.5"/>
   <link name="chassis">
-    <origin xyz = "0.0 0.0 0.055"/>
-    <visual>
-      <geometry>
-        <box size = "0.13 0.12 0.08"/>
-      </geometry>
-    </visual>
-    <collision>
-      <geometry>
-        <box size = "0.13 0.12 0.08"/>
+    <origin xyz="0.0 0.0 0.055"/>
+    <visual>
+      <geometry>
+        <box size="${c_len_x} ${c_len_y} ${c_len_z}"/>
+      </geometry>
+    </visual>
+    <collision>
+      <geometry>
+        <box size="${c_len_x} ${c_len_y} ${c_len_z}"/>
+      </geometry>
+    </collision>
+    <inertial>
+      <origin xyz="0.0 0.0 0.0"/>
+      <mass value="${c_mass}"/>
+      <inertia ixx="${(c_mass/12) * (c_len_y*c_len_y + c_len_z*c_len_z)}" ixy="0.0" ixz="0" iyy="${(c_mass/12) * (c_len_x*c_len_x + c_len_z*c_len_z)}" iyz="0.0" izz="${(c_mass/12) * (c_len_y*c_len_y + c_len_x*c_len_x)}"/>
+    </inertial>
+  </link>
+  <!-- Variables for battery -->
+  <xacro:property name="b_len_x" value="0.145"/>
+  <xacro:property name="b_len_y" value="0.065"/>
+  <xacro:property name="b_len_z" value="0.015"/>
+  <xacro:property name="b_mass" value="0.23"/>
+  <link name="battery">
+    <origin xyz="0.0 0.0 0.0"/>
+    <visual>
+      <geometry>
+        <box size="${b_len_x} ${b_len_y} ${b_len_z}"/>
+      </geometry>
+    </visual>
+    <collision>
+      <geometry>
+        <box size="${b_len_x} ${b_len_y} ${b_len_z}"/>
+      </geometry>
+    </collision>
+    <inertial>
+      <origin xyz="0.0 0.0 0.0"/>
+      <mass value="${b_mass}"/>
+      <inertia ixx="${(b_mass/12) * (b_len_y*b_len_y + b_len_z*b_len_z)}" ixy="0.0" ixz="0" iyy="${(b_mass/12) * (b_len_x*b_len_x + b_len_z*b_len_z)}" iyz="0.0" izz="${(b_mass/12) * (b_len_y*b_len_y + b_len_x*b_len_x)}"/>
+    </inertial>
+  </link>
+  <!-- Variables for wheels -->
+  <xacro:property name="w_rad" value="0.0325"/>
+  <xacro:property name="w_len" value="0.025"/>
+  <xacro:property name="w_mass" value="0.03"/>
+  <link name="front_left_wheel">
+    <visual>
+      <origin xyz="0.0 0.0125 0.0" rpy="1.5708 0 0"/>
+      <geometry>
+        <cylinder radius="${w_rad}" length="${w_len}"/>
+      </geometry>
+    </visual>
+    <collision>
+      <origin xyz="0.0 0.0125 0.0" rpy="1.5708 0 0"/>
+      <geometry>
+        <cylinder radius="${w_rad}" length="${w_len}"/>
       </geometry>
     </collision>
     <inertial>
       <origin xyz="0.0 0.0125 0.0"/>
-      <mass value="0.500"/>
-      <inertia ixx="0.00009565" ixy="0.0" ixz="0" iyy="0.0003999" iyz="0.0" izz="0.0004892"/>
-    </inertial>
-  </link>
-  <link name="battery">
-    <origin xyz = "0.0 0.0 0.0"/>
-    <visual>
-      <geometry>
-        <box size = "0.145 0.065 0.015"/>
-      </geometry>
-    </visual>
-    <collision>
-      <geometry>
-        <box size = "0.145 0.065 0.015"/>
-      </geometry>
-    </collision>
-    <inertial>
-      <origin xyz = "0.0 0.0 0.0"/>
-      <mass value="0.230"/>
-      <inertia ixx="0.00009435" ixy="0.0" ixz="0" iyy="0.00001117" iyz="0.0" izz="0.0000148"/>
-    </inertial>
-  </link>
-  <link name="front_left_wheel">
-    <visual>
-      <origin xyz="0.0 0.0125 0.0" rpy="1.5708 0 0"/>
-      <geometry>
-        <cylinder radius="0.0325" length="0.025"/>
-      </geometry>
-    </visual>
-    <collision>
-      <origin xyz="0.0 0.0125 0.0" rpy="1.5708 0 0"/>
-      <geometry>
-        <cylinder radius="0.0325" length="0.025"/>
+      <mass value="${w_mass}"/>
+      <inertia ixx="${(w_mass/12) * (3*w_rad*w_rad + w_len*w_len)}" ixy="0.0" ixz="0" iyy="${(w_mass/2) * (w_rad*w_rad)}" iyz="0.0" izz="${(w_mass/12) * (3*w_rad*w_rad + w_len*w_len)}"/>
+    </inertial>
+  </link>
+  <link name="front_right_wheel">
+    <visual>
+      <origin xyz="0.0 -0.0125 0.0" rpy="1.5708 0 0"/>
+      <geometry>
+        <cylinder radius="${w_rad}" length="${w_len}"/>
+      </geometry>
+    </visual>
+    <collision>
+      <origin xyz="0.0 -0.0125 0.0" rpy="1.5708 0 0"/>
+      <geometry>
+        <cylinder radius="${w_rad}" length="${w_len}"/>
+      </geometry>
+    </collision>
+    <inertial>
+      <origin xyz="0.0 -0.0125 0.0"/>
+      <mass value="${w_mass}"/>
+      <inertia ixx="${(w_mass/12) * (3*w_rad*w_rad + w_len*w_len)}" ixy="0.0" ixz="0" iyy="${(w_mass/2) * (w_rad*w_rad)}" iyz="0.0" izz="${(w_mass/12) * (3*w_rad*w_rad + w_len*w_len)}"/>
+    </inertial>
+  </link>
+  <link name="rear_left_wheel">
+    <visual>
+      <origin xyz="0.0 0.0125 0.0" rpy="1.5708 0 0"/>
+      <geometry>
+        <cylinder radius="${w_rad}" length="${w_len}"/>
+      </geometry>
+    </visual>
+    <collision>
+      <origin xyz="0.0 0.0125 0.0" rpy="1.5708 0 0"/>
+      <geometry>
+        <cylinder radius="${w_rad}" length="${w_len}"/>
       </geometry>
     </collision>
     <inertial>
       <origin xyz="0.0 0.0125 0.0"/>
-      <mass value="0.03"/>
-      <inertia ixx="0.00001044" ixy="0.0" ixz="0" iyy="0.00001767" iyz="0.0" izz="0.00001044"/>
-    </inertial>
-  </link>
-  <link name="front_right_wheel">
-    <visual>
-      <origin xyz="0.0 -0.0125 0.0" rpy="1.5708 0 0"/>
-      <geometry>
-        <cylinder radius="0.0325" length="0.025"/>
-      </geometry>
-    </visual>
-    <collision>
-      <origin xyz="0.0 -0.0125 0.0" rpy="1.5708 0 0"/>
-      <geometry>
-        <cylinder radius="0.0325" length="0.025"/>
+      <mass value="${w_mass}"/>
+      <inertia ixx="${(w_mass/12) * (3*w_rad*w_rad + w_len*w_len)}" ixy="0.0" ixz="0" iyy="${(w_mass/2) * (w_rad*w_rad)}" iyz="0.0" izz="${(w_mass/12) * (3*w_rad*w_rad + w_len*w_len)}"/>
+    </inertial>
+  </link>
+  <link name="rear_right_wheel">
+    <visual>
+      <origin xyz="0.0 -0.0125 0.0" rpy="1.5708 0 0"/>
+      <geometry>
+        <cylinder radius="${w_rad}" length="${w_len}"/>
+      </geometry>
+    </visual>
+    <collision>
+      <origin xyz="0.0 -0.0125 0.0" rpy="1.5708 0 0"/>
+      <geometry>
+        <cylinder radius="${w_rad}" length="${w_len}"/>
       </geometry>
     </collision>
     <inertial>
       <origin xyz="0.0 -0.0125 0.0"/>
-      <mass value="0.03"/>
-      <inertia ixx="0.00001044" ixy="0.0" ixz="0" iyy="0.00001767" iyz="0.0" izz="0.00001044"/>
-    </inertial>
-  </link>
-  <link name="rear_left_wheel">
-    <visual>
-      <origin xyz="0.0 0.0125 0.0" rpy="1.5708 0 0"/>
-      <geometry>
-        <cylinder radius="0.0325" length="0.025"/>
-      </geometry>
-    </visual>
-    <collision>
-      <origin xyz="0.0 0.0125 0.0" rpy="1.5708 0 0"/>
-      <geometry>
-        <cylinder radius="0.0325" length="0.025"/>
-      </geometry>
-    </collision>
-    <inertial>
-      <origin xyz="0.0 0.0125 0.0"/>
-      <mass value="0.03"/>
-      <inertia ixx="0.00001044" ixy="0.0" ixz="0" iyy="0.00001767" iyz="0.0" izz="0.00001044"/>
-    </inertial>
-  </link>
-  <link name="rear_right_wheel">
-    <visual>
-      <origin xyz="0.0 -0.0125 0.0" rpy="1.5708 0 0"/>
-      <geometry>
-        <cylinder radius="0.0325" length="0.025"/>
-      </geometry>
-    </visual>
-    <collision>
-      <origin xyz="0.0 -0.0125 0.0" rpy="1.5708 0 0"/>
-      <geometry>
-        <cylinder radius="0.0325" length="0.025"/>
-      </geometry>
-    </collision>
-    <inertial>
-      <origin xyz="0.0 -0.0125 0.0"/>
-      <mass value="0.03"/>
-      <inertia ixx="0.00001044" ixy="0.0" ixz="0" iyy="0.00001767" iyz="0.0" izz="0.00001044"/>
-    </inertial>
-  </link>
-  <joint name = "battery_mount" type="fixed">
-    <parent link = "chassis"/>
-    <child link = "battery"/>
-    <origin xyz = "0.015 0.0 0.0475"/>
-  </joint>
-  <joint name = "rear_right_axle" type="continuous">
-    <parent link = "chassis"/>
-    <child link = "rear_right_wheel"/>
-    <origin xyz = "-0.05 -0.06 -0.02"/>
-    <axis xyz = "0 1 0" />
-    <limit effort = "0.0784532" velocity="1.55"/>
-    <dynamics friction="0.04"/>
-  </joint>
-  <joint name = "rear_left_axle" type="continuous">
-    <parent link = "chassis"/>
-    <child link = "rear_left_wheel"/>
-    <origin xyz = "-0.05 0.06 -0.02"/>
-    <axis xyz = "0 1 0" />
-    <limit effort = "0.0784532" velocity="1.55"/>
-    <dynamics friction="0.04"/>
-  </joint>
-  <joint name = "front_left_axle" type="continuous">
-    <parent link = "chassis"/>
-    <child link = "front_left_wheel"/>
-    <origin xyz = "0.03 0.06 -0.02"/>
-    <axis xyz = "0 1 0" />
-    <limit effort = "0.0784532" velocity="1.55"/>
-    <dynamics friction="0.04"/>
-  </joint>
-  <joint name = "front_right_axle" type="continuous">
-    <parent link = "chassis"/>
-    <child link = "front_right_wheel"/>
-    <origin xyz = "0.03 -0.06 -0.02"/>
-    <axis xyz = "0 1 0" />
-    <limit effort = "0.0784532" velocity="1.55"/>
+      <mass value="${w_mass}"/>
+      <inertia ixx="${(w_mass/12) * (3*w_rad*w_rad + w_len*w_len)}" ixy="0.0" ixz="0" iyy="${(w_mass/2) * (w_rad*w_rad)}" iyz="0.0" izz="${(w_mass/12) * (3*w_rad*w_rad + w_len*w_len)}"/>
+    </inertial>
+  </link>
+  <joint name="battery_mount" type="fixed">
+    <parent link="chassis"/>
+    <child link="battery"/>
+    <origin xyz="0.015 0.0 0.0475"/>
+  </joint>
+  <joint name="rear_right_axle" type="continuous">
+    <parent link="chassis"/>
+    <child link="rear_right_wheel"/>
+    <origin xyz="-0.05 -0.06 -0.02"/>
+    <axis xyz="0 1 0" />
+    <limit effort="0.0784532" velocity="1.55"/>
+    <dynamics friction="0.04"/>
+  </joint>
+  <joint name="rear_left_axle" type="continuous">
+    <parent link="chassis"/>
+    <child link="rear_left_wheel"/>
+    <origin xyz="-0.05 0.06 -0.02"/>
+    <axis xyz="0 1 0" />
+    <limit effort="0.0784532" velocity="1.55"/>
+    <dynamics friction="0.04"/>
+  </joint>
+  <joint name="front_left_axle" type="continuous">
+    <parent link="chassis"/>
+    <child link="front_left_wheel"/>
+    <origin xyz="0.03 0.06 -0.02"/>
+    <axis xyz="0 1 0" />
+    <limit effort="0.0784532" velocity="1.55"/>
+    <dynamics friction="0.04"/>
+  </joint>
+  <joint name="front_right_axle" type="continuous">
+    <parent link="chassis"/>
+    <child link="front_right_wheel"/>
+    <origin xyz="0.03 -0.06 -0.02"/>
+    <axis xyz="0 1 0" />
+    <limit effort="0.0784532" velocity="1.55"/>
     <dynamics friction="0.04"/>
   </joint>
