Commit message: Working by adding masses

File: urdf/adeept_awr.urdf (robot description, URDF)
Before this commit: robot adeept_awr, 6 links, 5 joints
Links:
- removed link base
- link chassis: mass None -> 0.500
Joints:
- removed joint base_to_chassis

Commit message: added low friction to wheels

File: urdf/adeept_awr.urdf (robot description, URDF)
Before this commit: robot adeept_awr, 5 links, 4 joints
Joints:
- joint front_left_axle: limit (none) -> effort=0.0784532 velocity=1.55
- joint front_right_axle: limit (none) -> effort=0.0784532 velocity=1.55
- joint rear_left_axle: limit (none) -> effort=0.0784532 velocity=1.55
- joint rear_right_axle: limit (none) -> effort=0.0784532 velocity=1.55

Commit message: battery validated

File: urdf/adeept_awr.urdf (robot description, URDF)
Before this commit: robot adeept_awr, 5 links, 4 joints
Links:
- added link battery, mass 0.230; collision box size=0.145 0.065 0.015; visual box size=0.145 0.065 0.015
Joints:
- added joint battery_mount: type fixed, parent chassis, child battery, origin xyz=0.015 0.0 0.0475

Commit message: Add placeholder virtual camera

File: urdf/adeept_awr.urdf (robot description, URDF)
Before this commit: robot adeept_awr, 6 links, 5 joints
Links:
- added link camera_link, mass 1e-6; collision box size=1e-6 1e-6 1e-6; visual box size=1e-6 1e-6 1e-6
Joints:
- added joint camera_joint: type fixed, parent chassis, child camera_link, origin xyz=0.07 0.0 0.03 rpy=0 0 0
